File: gameboy-mbc0/plcc-socket-programmer.kicad_pcb (KiCad board)
At the start: 2 copper layers, 43.2 x 32.3 mm, 4 parts, among them P1 CONN_01X32, U1 SST39SF010

Commit message: adding .pro files and pcb updates
Parts:
- moved C1 3.81 mm to (129.3, 121.2), turned to 90 degrees
- moved C2 1.52 mm to (133.3, 120.1), turned to 90 degrees
Routing:
- net VCC: track 41.1 -> 42.3 mm
- net GND: track 110.3 -> 109.6 mm
Changed lines of the file:
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@@
   (general
     (links 34)
-    (no_connects 0)
+    (no_connects 1)
     (area 119.38 115.062 167.894001 150.368001)
     (thickness 1.6)
     (drawings 4)
-    (tracks 220)
+    (tracks 223)
     (zones 0)
     (modules 4)
@@
   )
   (module Capacitors_Tantalum_SMD:Tantalum_Case-R_EIA-2012-12_Hand (layer F.Cu)
-    (at 132.334 123.444 270)
+    (at 129.286 121.158 90)
     (descr "Tantalum capacitor, Case R, EIA 2012-12, 2.0x1.3x1.2mm, Hand soldering footprint")
     (tags "capacitor tantalum smd")
     (attr smd)
-    (fp_text reference C1 (at 0 -2.4 270) (layer F.SilkS)
+    (fp_text reference C1 (at 0 -2.4 90) (layer F.SilkS)
       (effects (font (size 1 1) (thickness 0.15)))
     )
-    (fp_text value 10uF (at 0 2.4 270) (layer F.Fab)
+    (fp_text value 10uF (at 0 2.4 90) (layer F.Fab)
       (effects (font (size 1 1) (thickness 0.15)))
     )
@@
     (fp_line (start -3.3 1.15) (end 1 1.15) (layer F.SilkS) (width 0.15))
     (fp_line (start -3.3 -1.15) (end -3.3 1.15) (layer F.SilkS) (width 0.15))
-    (pad 1 smd rect (at -1.7 0 270) (size 2.6 1.8) (layers F.Cu F.Mask)
+    (pad 1 smd rect (at -1.7 0 90) (size 2.6 1.8) (layers F.Cu F.Mask)
       (net 1 VCC))
-    (pad 2 smd rect (at 1.7 0 270) (size 2.6 1.8) (layers F.Cu F.Mask)
+    (pad 2 smd rect (at 1.7 0 90) (size 2.6 1.8) (layers F.Cu F.Mask)
       (net 32 GND))
     (model Capacitors_Tantalum_SMD.3dshapes/Tantalum_Case-R_EIA-2012-12.wrl
@@
   )
   (module Capacitors_SMD:C_0805_HandSoldering (layer F.Cu)
-    (at 134.874 120.142 270)
+    (at 133.35 120.142 90)
     (descr "Capacitor SMD 0805, hand soldering")
     (tags "capacitor 0805")
     (attr smd)
-    (fp_text reference C2 (at 0 -2.1 270) (layer F.SilkS)
+    (fp_text reference C2 (at 0 -2.1 90) (layer F.SilkS)
       (effects (font (size 1 1) (thickness 0.15)))
     )
-    (fp_text value 0.1uF (at 0 2.1 270) (layer F.Fab)
+    (fp_text value 0.1uF (at 0 2.1 90) (layer F.Fab)
       (effects (font (size 1 1) (thickness 0.15)))
     )
@@
     (fp_line (start 0.5 -0.85) (end -0.5 -0.85) (layer F.SilkS) (width 0.15))
     (fp_line (start -0.5 0.85) (end 0.5 0.85) (layer F.SilkS) (width 0.15))
-    (pad 1 smd rect (at -1.25 0 270) (size 1.5 1.25) (layers F.Cu F.Mask)
+    (pad 1 smd rect (at -1.25 0 90) (size 1.5 1.25) (layers F.Cu F.Mask)
       (net 1 VCC))
-    (pad 2 smd rect (at 1.25 0 270) (size 1.5 1.25) (layers F.Cu F.Mask)
+    (pad 2 smd rect (at 1.25 0 90) (size 1.5 1.25) (layers F.Cu F.Mask)
       (net 32 GND))
     (model Capacitors_SMD.3dshapes/C_0805_HandSoldering.wrl
@@
   (gr_line (start 123.19 148.59) (end 166.37 148.59) (angle 90) (layer Edge.Cuts) (width 0.15))
   (gr_line (start 166.37 148.59) (end 166.37 116.332) (angle 90) (layer Edge.Cuts) (width 0.15))
-  (segment (start 125.73 143.51) (end 125.73 128.348) (width 0.4064) (layer F.Cu) (net 1))
-  (segment (start 125.73 128.348) (end 132.334 121.744) (width 0.4064) (layer F.Cu) (net 1))
-  (segment (start 132.334 121.744) (end 132.334 121.432) (width 0.4064) (layer F.Cu) (net 1))
-  (segment (start 132.334 121.432) (end 134.874 118.892) (width 0.4064) (layer F.Cu) (net 1))
-  (segment (start 146.05 119.38) (end 146.05 120.904) (width 0.4064) (layer F.Cu) (net 1))
+  (segment (start 133.35 121.392) (end 130.752 121.392) (width 0.4064) (layer F.Cu) (net 1) (status 400000))
+  (segment (start 125.73 128.348) (end 125.73 143.51) (width 0.4064) (layer F.Cu) (net 1))
+  (segment (start 125.73 126.414) (end 125.73 128.348) (width 0.4064) (layer F.Cu) (net 1))
+  (segment (start 130.752 121.392) (end 125.73 126.414) (width 0.4064) (layer F.Cu) (net 1))
+  (segment (start 139.7 118.872) (end 135.87 118.872) (width 0.4064) (layer F.Cu) (net 1))
+  (segment (start 146.05 120.904) (end 146.05 119.38) (width 0.4064) (layer F.Cu) (net 1))
   (segment (start 145.542 118.872) (end 146.05 119.38) (width 0.4064) (layer F.Cu) (net 1))
-  (segment (start 135.128 118.872) (end 145.542 118.872) (width 0.4064) (layer F.Cu) (net 1))
+  (segment (start 139.7 118.872) (end 145.542 118.872) (width 0.4064) (layer F.Cu) (net 1))
+  (segment (start 135.87 118.872) (end 133.35 121.392) (width 0.4064) (layer F.Cu) (net 1) (status 800000))
   (segment (start 128.27 143.51) (end 136.906 134.874) (width 0.2032) (layer B.Cu) (net 3))
   (segment (start 147.32 124.714) (end 148.59 123.444) (width 0.2032) (layer F.Cu) (net 3))
@@
   (segment (start 161.29 143.51) (end 161.036 143.51) (width 0.2032) (layer F.Cu) (net 29))
   (segment (start 161.036 143.51) (end 151.13 133.604) (width 0.2032) (layer F.Cu) (net 29))
-  (segment (start 128.524 127.762) (end 129.716 127.762) (width 0.2032) (layer F.Cu) (net 32))
-  (segment (start 134.874 122.604) (end 134.874 121.392) (width 0.2032) (layer F.Cu) (net 32))
-  (segment (start 129.716 127.762) (end 134.874 122.604) (width 0.2032) (layer F.Cu) (net 32))
+  (segment (start 133.35 118.892) (end 129.852 118.892) (width 0.2032) (layer F.Cu) (net 32) (status C00000))
+  (segment (start 129.852 118.892) (end 129.286 119.458) (width 0.2032) (layer F.Cu) (net 32) (status C00000))
+  (segment (start 125.73 118.872) (end 128.7 118.872) (width 0.2032) (layer F.Cu) (net 32) (status 800000))
+  (segment (start 128.7 118.872) (end 129.286 119.458) (width 0.2032) (layer F.Cu) (net 32) (status C00000))
   (via (at 128.524 137.414) (size 0.762) (drill 0.381) (layers F.Cu B.Cu) (net 32))
   (segment (start 128.524 132.588) (end 128.524 137.414) (width 0.2032) (layer B.Cu) (net 32))
   (via (at 128.524 132.588) (size 0.762) (drill 0.381) (layers F.Cu B.Cu) (net 32))
-  (segment (start 128.524 127.762) (end 128.524 132.588) (width 0.2032) (layer F.Cu) (net 32))
-  (via (at 128.524 127.762) (size 0.762) (drill 0.381) (layers F.Cu B.Cu) (net 32))
-  (segment (start 125.73 124.968) (end 128.524 127.762) (width 0.2032) (layer B.Cu) (net 32))
-  (via (at 125.73 124.968) (size 0.762) (drill 0.381) (layers F.Cu B.Cu) (net 32))
-  (segment (start 131.826 118.872) (end 125.73 124.968) (width 0.2032) (layer F.Cu) (net 32))
-  (via (at 131.826 118.872) (size 0.762) (drill 0.381) (layers F.Cu B.Cu) (net 32))
+  (segment (start 128.524 126.492) (end 128.524 132.588) (width 0.2032) (layer F.Cu) (net 32))
+  (via (at 128.524 126.492) (size 0.762) (drill 0.381) (layers F.Cu B.Cu) (net 32))
+  (segment (start 125.73 123.698) (end 128.524 126.492) (width 0.2032) (layer B.Cu) (net 32))
+  (via (at 125.73 123.698) (size 0.762) (drill 0.381) (layers F.Cu B.Cu) (net 32))
+  (segment (start 125.73 118.872) (end 125.73 123.698) (width 0.2032) (layer F.Cu) (net 32))
+  (via (at 125.73 118.872) (size 0.762) (drill 0.381) (layers F.Cu B.Cu) (net 32))
   (segment (start 143.51 120.904) (end 141.478 118.872) (width 0.2032) (layer B.Cu) (net 32))
-  (segment (start 141.478 118.872) (end 131.826 118.872) (width 0.2032) (layer B.Cu) (net 32))
+  (segment (start 141.478 118.872) (end 125.73 118.872) (width 0.2032) (layer B.Cu) (net 32))
   (segment (start 143.51 125.984) (end 143.51 128.524) (width 0.2032) (layer F.Cu) (net 32))
   (via (at 146.05 131.064) (size 0.762) (drill 0.381) (layers F.Cu B.Cu) (net 32))
@@
   (segment (start 163.83 146.05) (end 162.56 144.78) (width 0.2032) (layer F.Cu) (net 32))
   (segment (start 145.542 118.872) (end 143.51 120.904) (width 0.2032) (layer B.Cu) (net 32))
-  (segment (start 153.67 118.872) (end 145.542 118.872) (width 0.2032) (layer B.Cu) (net 32))
-  (via (at 153.67 118.872) (size 0.762) (drill 0.381) (layers F.Cu B.Cu) (net 32))
-  (segment (start 156.21 121.412) (end 153.67 118.872) (width 0.2032) (layer F.Cu) (net 32))
-  (via (at 156.21 121.412) (size 0.762) (drill 0.381) (layers F.Cu B.Cu) (net 32))
-  (segment (start 159.258 124.46) (end 156.21 121.412) (width 0.2032) (layer B.Cu) (net 32))
-  (via (at 159.258 124.46) (size 0.762) (drill 0.381) (layers F.Cu B.Cu) (net 32))
-  (segment (start 162.56 127.762) (end 159.258 124.46) (width 0.2032) (layer F.Cu) (net 32))
-  (via (at 162.56 127.762) (size 0.762) (drill 0.381) (layers F.Cu B.Cu) (net 32))
-  (segment (start 162.56 132.08) (end 162.56 127.762) (width 0.2032) (layer B.Cu) (net 32))
-  (via (at 162.56 132.08) (size 0.762) (drill 0.381) (layers F.Cu B.Cu) (net 32))
-  (segment (start 162.56 136.652) (end 162.56 132.08) (width 0.2032) (layer F.Cu) (net 32))
+  (segment (start 149.098 118.872) (end 145.542 118.872) (width 0.2032) (layer B.Cu) (net 32))
+  (via (at 149.098 118.872) (size 0.762) (drill 0.381) (layers F.Cu B.Cu) (net 32))
+  (segment (start 153.67 123.444) (end 149.098 118.872) (width 0.2032) (layer F.Cu) (net 32))
+  (via (at 153.67 123.444) (size 0.762) (drill 0.381) (layers F.Cu B.Cu) (net 32))
+  (segment (start 157.226 127) (end 153.67 123.444) (width 0.2032) (layer B.Cu) (net 32))
+  (via (at 157.226 127) (size 0.762) (drill 0.381) (layers F.Cu B.Cu) (net 32))
+  (segment (start 160.528 130.302) (end 157.226 127) (width 0.2032) (layer F.Cu) (net 32))
+  (via (at 160.528 130.302) (size 0.762) (drill 0.381) (layers F.Cu B.Cu) (net 32))
+  (segment (start 162.56 132.334) (end 160.528 130.302) (width 0.2032) (layer B.Cu) (net 32))
+  (via (at 162.56 132.334) (size 0.762) (drill 0.381) (layers F.Cu B.Cu) (net 32))
+  (segment (start 162.56 136.652) (end 162.56 132.334) (width 0.2032) (layer F.Cu) (net 32))
   (via (at 162.56 136.652) (size 0.762) (drill 0.381) (layers F.Cu B.Cu) (net 32))
   (segment (start 162.56 141.224) (end 162.56 136.652) (width 0.2032) (layer B.Cu) (net 32))
